Commit message: laser reverse

File: sentry_description/urdf/sentry_description.gazebo.xacro (robot description, xacro)
@@ -113,5 +113,6 @@
   </link>
   <joint name="laser_static" type="fixed">
-    <origin xyz="0 0 0.4" rpy="0 0 0" />
+    <origin xyz="0 0 0.4" rpy="3.1415926 0 0" />
+    <!-- <origin xyz="0 0 0.4" rpy="0 0 0" /> -->
     <parent link="arm" />
     <child link="livox_laser" />
@@ -209,9 +210,9 @@
       <update_rate>500</update_rate>
       <visualize>true</visualize>
-      <topic>imu_at_camera</topic>
+      <topic>imu</topic>
       <plugin name="imu_plugin" filename="libgazebo_ros_imu_sensor.so">
         <topicName>imu</topicName>
         <bodyName>livox_laser</bodyName>
-        <updateRateHZ>100.0</updateRateHZ>
+        <updateRateHZ>500.0</updateRateHZ>
         <gaussianNoise>0.0</gaussianNoise>
         <xyzOffset>0 0 0</xyzOffset>
